File: MPPT_Sensors.kicad_sch (KiCad schematic)
At the start: 22 parts, among them IC1 MAX22531AAP+, IC3 MCP6C26T-050E_LTY, IC4 BU7421SG-TR, IC5 MCP6C26T-050E_LTY, IC6 BU7421SG-TR

Commit message: Minor changes to connectors and amplifiers
Parts:
- removed R12, R13, R8, R9: R, symbol Device:R
- added D2, D4, D5, D6: SZESD5Z5.0T5G, symbol Device:D
Connections:
- net +3V3_HV: now also D2.1 (K), D4.1 (K), D5.1 (K), D6.1 (K)
- net Array_C: now also D4.2 (A)
- net Array_V: now also IC6.3 (IN-), D2.2 (A)
- net Battery_C: now also D5.2 (A)
- net Battery_V: now also IC4.3 (IN-), D6.2 (A)
Other:
- note added: "Isolated ADC"
- note added: "There aren't really isolated amplifiers on the market that let us achieve the desired granularity with a small shunt resistor, and with the single ended output needed to interface with the PSOM ADC. Therefore i chose to use a discrete, isolated ADC."
- note removed: "There aren't really isolated amplifiers on the market that let us achieve the desired granularity with a small shunt resistor, and with the single ended output needed to interface with the PSOM ADC. Therefore we probably need to use a discrete, isolated ADC."
- moved on the sheet: C13, C14, C15, IC1

Commit message: Fixed PSOM pinout, added 24v-3.3v iso supply, moved current sensing to low side
Parts:
- removed R2, R3: 10k, symbol Device:R
Connections:
- net Vref is gone; now on net HV_GND: IC3.1 (VREF), IC5.1 (VREF)
Other:
- note added: "No vref chip needed since tying ref to gnd."
